File: PMT9123_breakout.kicad_pcb (KiCad board)
At the start: 2 copper layers, 21 parts, among them P1 CONN_01X06, Q1 BSS138, Q2 BSS138, Q3 BSS138, Q4 BSS138, U1 MIC5365-1.8YC5, U2 PMT9123

Commit message: PCB done
Parts:
- added C6: 0.1u, Capacitors_SMD:C_0805, F.Cu at (131.2, 103.5)
- added MH1: MH, Mounting_Holes:MountingHole_2.2mm_M2_Pad_Via, F.Cu at (133.0, 92.0)
- added MH2: MH, Mounting_Holes:MountingHole_2.2mm_M2_Pad_Via, F.Cu at (133.0, 107.0)
- U2: footprint Housings_DFN_QFN:QFN-28-1EP_6x6mm_Pitch0.65mm -> aesora:PMT9123
- moved C5 43.4 mm to (138.5, 105.8), turned to 180 degrees
- moved R9 37.6 mm to (134.8, 103.5), turned to 180 degrees
- moved C3 20.0 mm to (139.0, 92.4), turned to 90 degrees
- moved C4 3.25 mm to (138.5, 103.5)
- moved U2 2.24 mm to (137.0, 98.5)
- moved R3 0.75 mm to (127.2, 99.5)
- moved R5 0.75 mm to (127.2, 103.5)
- moved R7 0.75 mm to (127.2, 107.5)
- moved C2 0.50 mm to (127.5, 91.5)
- moved R1 0.50 mm to (127.5, 95.5)
Routing:
- net +1V8: track 35.6 -> 60.1 mm, vias 0 -> 2
- net /SCL_LV: track 2.50 -> 15.8 mm
- net GND: track 7.45 -> 16.3 mm, vias 6 -> 13
- net Net-(R9-Pad1): track 0.00 -> 3.76 mm
- net Net-(U2-Pad19): track 12.0 -> 9.08 mm
- net /SDA_LV: track 11.6 -> 9.59 mm
- net /~MOT~_LV: track 12.5 -> 10.9 mm
- net Net-(C4-Pad1): track 6.87 -> 7.43 mm, vias 0 -> 2
- added copper zone on B.Cu, net GND
Other:
- board outline added: 28.6 x 21.5 mm
- board text added: "GND"
- board text added: "SCL"
- board text added: "SDA"
- board text added: "V1.0"
- board text added: "VCC"
- board text added: "www.aesora.de"
- board text added: "~MOT~"
- board text added: "~RST~"
