File: PMT9123_breakout.sch (KiCad schematic (older format))
At the start: 21 parts, among them P1 CONN_01X06, Q1 BSS138, Q2 BSS138, Q3 BSS138, Q4 BSS138, U1 MIC5365-1.8YC5, U2 PMT9123

Commit message: added missing footprints
Parts:
- R9: footprint (none) -> Resistors_SMD:R_0805_HandSoldering
- U2: footprint (none) -> Housings_DFN_QFN:QFN-28-1EP_6x6mm_Pitch0.65mm
Changed lines of the file:
@@
 F 0 "U2" H 3000 150 60  0000 C CNN
 F 1 "PMT9123" H 3000 2150 60  0000 C CNN
-F 2 "" H 3000 2100 60  0001 C CNN
+F 2 "Housings_DFN_QFN:QFN-28-1EP_6x6mm_Pitch0.65mm" H 3000 2100 60  0001 C CNN
 F 3 "" H 3000 2100 60  0001 C CNN
 	1    3000 2100
@@
 F 0 "R9" V 2330 3300 50  0000 C CNN
 F 1 "43" V 2250 3300 50  0000 C CNN
-F 2 "" V 2180 3300 50  0000 C CNN
+F 2 "Resistors_SMD:R_0805_HandSoldering" V 2180 3300 50  0001 C CNN
 F 3 "" H 2250 3300 50  0000 C CNN
 	1    2250 3300

Commit message: started pcb
Parts:
- C1, C2, C3, C4, C5: footprint Capacitors_SMD:C_0805_HandSoldering -> Capacitors_SMD:C_0805
- R1, R2, R3, R4, R5, R6, R7, R8, R9: footprint Resistors_SMD:R_0805_HandSoldering -> Resistors_SMD:R_0805
Changed lines of the file:
@@
 F 0 "R1" V 1180 1250 50  0000 C CNN
 F 1 "10k" V 1100 1250 50  0000 C CNN
-F 2 "Resistors_SMD:R_0805_HandSoldering" V 1030 1250 50  0001 C CNN
+F 2 "Resistors_SMD:R_0805" V 1030 1250 50  0001 C CNN
 F 3 "" H 1100 1250 50  0000 C CNN
 	1    1100 1250
@@
 F 0 "R2" V 1780 1250 50  0000 C CNN
 F 1 "10k" V 1700 1250 50  0000 C CNN
-F 2 "Resistors_SMD:R_0805_HandSoldering" V 1630 1250 50  0001 C CNN
+F 2 "Resistors_SMD:R_0805" V 1630 1250 50  0001 C CNN
 F 3 "" H 1700 1250 50  0000 C CNN
 	1    1700 1250
@@
 F 0 "R3" V 3080 1250 50  0000 C CNN
 F 1 "10k" V 3000 1250 50  0000 C CNN
-F 2 "Resistors_SMD:R_0805_HandSoldering" V 2930 1250 50  0001 C CNN
+F 2 "Resistors_SMD:R_0805" V 2930 1250 50  0001 C CNN
 F 3 "" H 3000 1250 50  0000 C CNN
 	1    3000 1250
@@
 F 0 "R4" V 3680 1250 50  0000 C CNN
 F 1 "10k" V 3600 1250 50  0000 C CNN
-F 2 "Resistors_SMD:R_0805_HandSoldering" V 3530 1250 50  0001 C CNN
+F 2 "Resistors_SMD:R_0805" V 3530 1250 50  0001 C CNN
 F 3 "" H 3600 1250 50  0000 C CNN
 	1    3600 1250
@@
 F 0 "R5" V 4980 1250 50  0000 C CNN
 F 1 "10k" V 4900 1250 50  0000 C CNN
-F 2 "Resistors_SMD:R_0805_HandSoldering" V 4830 1250 50  0001 C CNN
+F 2 "Resistors_SMD:R_0805" V 4830 1250 50  0001 C CNN
 F 3 "" H 4900 1250 50  0000 C CNN
 	1    4900 1250
@@
 F 0 "R6" V 5580 1250 50  0000 C CNN
 F 1 "10k" V 5500 1250 50  0000 C CNN
-F 2 "Resistors_SMD:R_0805_HandSoldering" V 5430 1250 50  0001 C CNN
+F 2 "Resistors_SMD:R_0805" V 5430 1250 50  0001 C CNN
 F 3 "" H 5500 1250 50  0000 C CNN
 	1    5500 1250
@@
 F 0 "R7" V 6880 1250 50  0000 C CNN
 F 1 "10k" V 6800 1250 50  0000 C CNN
-F 2 "Resistors_SMD:R_0805_HandSoldering" V 6730 1250 50  0001 C CNN
+F 2 "Resistors_SMD:R_0805" V 6730 1250 50  0001 C CNN
 F 3 "" H 6800 1250 50  0000 C CNN
 	1    6800 1250
@@
 F 0 "R8" V 7480 1250 50  0000 C CNN
 F 1 "10k" V 7400 1250 50  0000 C CNN
-F 2 "Resistors_SMD:R_0805_HandSoldering" V 7330 1250 50  0001 C CNN
+F 2 "Resistors_SMD:R_0805" V 7330 1250 50  0001 C CNN
 F 3 "" H 7400 1250 50  0000 C CNN
 	1    7400 1250
@@
 F 0 "C2" H 10225 1550 50  0000 L CNN
 F 1 "4.7u" H 10225 1350 50  0000 L CNN
-F 2 "Capacitors_SMD:C_0805_HandSoldering" H 10238 1300 50  0001 C CNN
+F 2 "Capacitors_SMD:C_0805" H 10238 1300 50  0001 C CNN
 F 3 "" H 10200 1450 50  0000 C CNN
 	1    10200 1450
@@
 F 0 "C1" H 8925 1550 50  0000 L CNN
 F 1 "4.7u" H 8925 1350 50  0000 L CNN
-F 2 "Capacitors_SMD:C_0805_HandSoldering" H 8938 1300 50  0001 C CNN
+F 2 "Capacitors_SMD:C_0805" H 8938 1300 50  0001 C CNN
 F 3 "" H 8900 1450 50  0000 C CNN
 	1    8900 1450
@@
 F 0 "R9" V 2330 3300 50  0000 C CNN
 F 1 "43" V 2250 3300 50  0000 C CNN
-F 2 "Resistors_SMD:R_0805_HandSoldering" V 2180 3300 50  0001 C CNN
+F 2 "Resistors_SMD:R_0805" V 2180 3300 50  0001 C CNN
 F 3 "" H 2250 3300 50  0000 C CNN
 	1    2250 3300
@@
 F 0 "C5" H 2175 2900 50  0000 L CNN
 F 1 "4.7u" H 2175 2700 50  0000 L CNN
-F 2 "Capacitors_SMD:C_0805_HandSoldering" H 2188 2650 50  0001 C CNN
+F 2 "Capacitors_SMD:C_0805" H 2188 2650 50  0001 C CNN
 F 3 "" H 2150 2800 50  0000 C CNN
 	1    2150 2800
@@
 F 0 "C4" H 2175 2600 50  0000 L CNN
 F 1 "0.1u" H 2175 2400 50  0000 L CNN
-F 2 "Capacitors_SMD:C_0805_HandSoldering" H 2188 2350 50  0001 C CNN
+F 2 "Capacitors_SMD:C_0805" H 2188 2350 50  0001 C CNN
 F 3 "" H 2150 2500 50  0000 C CNN
 	1    2150 2500
@@
 F 0 "C3" H 2175 2300 50  0000 L CNN
 F 1 "0.1u" H 2175 2100 50  0000 L CNN
-F 2 "Capacitors_SMD:C_0805_HandSoldering" H 2188 2050 50  0001 C CNN
+F 2 "Capacitors_SMD:C_0805" H 2188 2050 50  0001 C CNN
 F 3 "" H 2150 2200 50  0000 C CNN
 	1    2150 2200

Commit message: PCB done
Parts:
- added C6: 0.1u, Capacitors_SMD:C_0805, symbol C
- added MH1, MH2: MH, Mounting_Holes:MountingHole_2.2mm_M2_Pad_Via, symbol CONN_01X01
- U2: footprint Housings_DFN_QFN:QFN-28-1EP_6x6mm_Pitch0.65mm -> aesora:PMT9123
Connections:
- net +1V8: now also C6.1
- net GND: now also C6.2, MH1.1 (P1), MH2.1 (P1)
Changed lines of the file:
@@
 	9650 1600 9650 1550
-$Comp
-L PMT9123 U2
-U 1 1 58349186
-P 3000 2100
-F 0 "U2" H 3000 150 60  0000 C CNN
-F 1 "PMT9123" H 3000 2150 60  0000 C CNN
-F 2 "Housings_DFN_QFN:QFN-28-1EP_6x6mm_Pitch0.65mm" H 3000 2100 60  0001 C CNN
-F 3 "" H 3000 2100 60  0001 C CNN
-	1    3000 2100
-	1    0    0    -1
-$EndComp
 $Comp
 L +1V8 #PWR016
@@
 L +1V8 #PWR017
 U 1 1 583498CE
-P 2100 3300
-F 0 "#PWR017" H 2100 3150 50  0001 C CNN
-F 1 "+1V8" H 2100 3440 50  0000 C CNN
-F 2 "" H 2100 3300 50  0000 C CNN
-F 3 "" H 2100 3300 50  0000 C CNN
-	1    2100 3300
+P 2050 3250
+F 0 "#PWR017" H 2050 3100 50  0001 C CNN
+F 1 "+1V8" H 2050 3390 50  0000 C CNN
+F 2 "" H 2050 3250 50  0000 C CNN
+F 3 "" H 2050 3250 50  0000 C CNN
+	1    2050 3250
 	1    0    0    -1
 $EndComp
@@
 L GND #PWR020
 U 1 1 5834C7C0
-P 900 3900
-F 0 "#PWR020" H 900 3650 50  0001 C CNN
-F 1 "GND" H 900 3750 50  0000 C CNN
-F 2 "" H 900 3900 50  0000 C CNN
-F 3 "" H 900 3900 50  0000 C CNN
-	1    900  3900
+P 5000 2600
+F 0 "#PWR020" H 5000 2350 50  0001 C CNN
+F 1 "GND" H 5000 2450 50  0000 C CNN
+F 2 "" H 5000 2600 50  0000 C CNN
+F 3 "" H 5000 2600 50  0000 C CNN
+	1    5000 2600
 	1    0    0    -1
 $EndComp
@@
 L +5V #PWR021
 U 1 1 5834C80A
-P 900 3400
-F 0 "#PWR021" H 900 3250 50  0001 C CNN
-F 1 "+5V" H 900 3540 50  0000 C CNN
-F 2 "" H 900 3400 50  0000 C CNN
-F 3 "" H 900 3400 50  0000 C CNN
-	1    900  3400
+P 4700 2300
+F 0 "#PWR021" H 4700 2150 50  0001 C CNN
+F 1 "+5V" H 4700 2440 50  0000 C CNN
+F 2 "" H 4700 2300 50  0000 C CNN
+F 3 "" H 4700 2300 50  0000 C CNN
+	1    4700 2300
 	1    0    0    -1
 $EndComp
@@
 L PWR_FLAG #FLG022
 U 1 1 5834C880
-P 1200 3400
-F 0 "#FLG022" H 1200 3495 50  0001 C CNN
-F 1 "PWR_FLAG" H 1200 3580 50  0000 C CNN
-F 2 "" H 1200 3400 50  0000 C CNN
-F 3 "" H 1200 3400 50  0000 C CNN
-	1    1200 3400
+P 5000 2300
+F 0 "#FLG022" H 5000 2395 50  0001 C CNN
+F 1 "PWR_FLAG" H 5000 2480 50  0000 C CNN
+F 2 "" H 5000 2300 50  0000 C CNN
+F 3 "" H 5000 2300 50  0000 C CNN
+	1    5000 2300
 	1    0    0    -1
 $EndComp
@@
 L PWR_FLAG #FLG023
 U 1 1 5834C8BE
-P 900 3900
-F 0 "#FLG023" H 900 3995 50  0001 C CNN
-F 1 "PWR_FLAG" H 900 4080 50  0000 C CNN
-F 2 "" H 900 3900 50  0000 C CNN
-F 3 "" H 900 3900 50  0000 C CNN
-	1    900  3900
-	1    0    0    -1
-$EndComp
-Wire Wire Line
-	1200 3400 900  3400
+P 5000 2600
+F 0 "#FLG023" H 5000 2695 50  0001 C CNN
+F 1 "PWR_FLAG" H 5000 2780 50  0000 C CNN
+F 2 "" H 5000 2600 50  0000 C CNN
+F 3 "" H 5000 2600 50  0000 C CNN
+	1    5000 2600
+	1    0    0    -1
+$EndComp
+Wire Wire Line
+	5000 2300 4700 2300
+$Comp
+L PMT9123 U2
+U 1 1 5834A5DB
+P 3000 2100
+F 0 "U2" H 3000 150 60  0000 C CNN
+F 1 "PMT9123" H 3000 2150 60  0000 C CNN
+F 2 "aesora:PMT9123" H 3000 2100 60  0001 C CNN
+F 3 "" H 3000 2100 60  0001 C CNN
+	1    3000 2100
+	1    0    0    -1
+$EndComp
+$Comp
+L C C6
+U 1 1 5834AAD9
+P 2050 3500
+F 0 "C6" H 2075 3600 50  0000 L CNN
+F 1 "0.1u" H 2075 3400 50  0000 L CNN
+F 2 "Capacitors_SMD:C_0805" H 2088 3350 50  0001 C CNN
+F 3 "" H 2050 3500 50  0000 C CNN
+	1    2050 3500
+	1    0    0    -1
+$EndComp
+Wire Wire Line
+	2050 3250 2050 3350
+Connection ~ 2050 3300
+$Comp
+L GND #PWR024
+U 1 1 5834ADE4
+P 2050 3650
+F 0 "#PWR024" H 2050 3400 50  0001 C CNN
+F 1 "GND" H 2050 3500 50  0000 C CNN
+F 2 "" H 2050 3650 50  0000 C CNN
+F 3 "" H 2050 3650 50  0000 C CNN
+	1    2050 3650
+	1    0    0    -1
+$EndComp
+Wire Wire Line
+	2100 3300 2050 3300
+$Comp
+L CONN_01X01 MH1
+U 1 1 5834B59D
+P 5000 3100
+F 0 "MH1" H 5000 3200 50  0000 C CNN
+F 1 "MH" V 5100 3100 50  0000 C CNN
+F 2 "Mounting_Holes:MountingHole_2.2mm_M2_Pad_Via" H 5000 3100 50  0001 C CNN
+F 3 "" H 5000 3100 50  0000 C CNN
+	1    5000 3100
+	1    0    0    -1
+$EndComp
+$Comp
+L CONN_01X01 MH2
+U 1 1 5834B818
+P 5000 3400
+F 0 "MH2" H 5000 3500 50  0000 C CNN
+F 1 "MH" V 5100 3400 50  0000 C CNN
+F 2 "Mounting_Holes:MountingHole_2.2mm_M2_Pad_Via" H 5000 3400 50  0001 C CNN
+F 3 "" H 5000 3400 50  0000 C CNN
+	1    5000 3400
+	1    0    0    -1
+$EndComp
+$Comp
+L GND #PWR025
+U 1 1 5834BB2E
+P 4800 3400
+F 0 "#PWR025" H 4800 3150 50  0001 C CNN
+F 1 "GND" H 4800 3250 50  0000 C CNN
+F 2 "" H 4800 3400 50  0000 C CNN
+F 3 "" H 4800 3400 50  0000 C CNN
+	1    4800 3400
+	1    0    0    -1
+$EndComp
+$Comp
+L GND #PWR026
+U 1 1 5834BB81
+P 4800 3100
+F 0 "#PWR026" H 4800 2850 50  0001 C CNN
+F 1 "GND" H 4800 2950 50  0000 C CNN
+F 2 "" H 4800 3100 50  0000 C CNN
+F 3 "" H 4800 3100 50  0000 C CNN
+	1    4800 3100
+	1    0    0    -1
+$EndComp
 $EndSCHEMATC
